Commit message: fix base_link yaw

File: simplebot_description/urdf/simplebot.urdf (robot description, URDF)
Before this commit: robot simplebot, 9 links, 8 joints
Joints:
- joint base_joint: origin xyz=0 0 0 rpy=0 0 0 -> xyz=0 0 0 rpy=0 0 -1.57
- joint lidar_joint: origin xyz=0 0.12 0.0125 rpy=0 0 1.57 -> xyz=0 0.12 0.0125 rpy=0 0 0

Commit message: add gmapping and fix urdf

File: simplebot_description/urdf/simplebot.urdf (robot description, URDF)
Before this commit: robot simplebot, 9 links, 8 joints
Joints:
- joint caster_ball_joint: origin xyz=0 0 -0.0225 rpy=0 0 1.57 -> xyz=0 0 -0.025 rpy=0 0 1.57

Commit message: move_baseひとまずgazeboで動いた（パラメーター適当）

File: simplebot_description/urdf/simplebot.urdf (robot description, URDF)
Before this commit: robot simplebot, 9 links, 8 joints
Joints:
- joint base_joint: origin xyz=0 0 0 rpy=0 0 -1.57 -> xyz=0 0 0.0535 rpy=0 0 -1.57
